File: room-pcb.kicad_sch (KiCad schematic)
At the start: 28 parts, among them J1 Conn_01x08, J2 Conn_01x02, J3 Conn_01x04, J4 Conn_01x05, U1 COZIR, U2 BH1750FVI-TR, U3 AHT20, U5 ESP32-C6_SUPERMINI_TH

Commit message: first order
Parts:
- removed D3: WS2812B, LED_SMD:LED_WS2812B-2020_PLCC4_2.0x2.0mm, symbol LED:WS2812B
- added J5, J6: Conn_01x04, Connector_PinHeader_2.54mm:PinHeader_1x04_P2.54mm_Vertical, symbol Connector_Generic:Conn_01x04
Connections:
- net +3.3V: now also J5.2 (Pin_2), J6.2 (Pin_2)
- net CS: no longer U5.8 (GPIO8)
- net GND: now also J5.1 (Pin_1), J6.1 (Pin_1)
- net EX2: now reaches U5.14 (GPIO14)
- net EX2: now also J5.4 (Pin_4)
- net EX3: now reaches U5.15 (GPIO15)
- net EX3: now also J6.3 (Pin_3)
- net EX4: now reaches U5.18 (GPIO18)
- net EX4: now also J6.4 (Pin_4)
- net EX1: now reaches U5.9 (GPIO9)
- net EX1: now also J5.3 (Pin_3)
- no-connect marks 12 -> 14
