File: room-pcb.kicad_sch (KiCad schematic)
At the start: 28 parts, among them J1 Conn_01x08, J2 Conn_01x02, J3 Conn_01x04, U1 COZIR, U2 BH1750FVI-TR, U3 AHT20, U4 LD2450, U5 ESP32-C6_SUPERMINI_TH

Commit message: new layout
Parts:
- removed U4: LD2450, ld2450:ld2450, symbol ld2450:ld2450
- added J4: Conn_01x05, Connector_PinHeader_1.27mm:PinHeader_1x05_P1.27mm_Vertical, symbol Connector_Generic:Conn_01x05
- C3, J1: now not fitted; now left out of the parts list
Connections:
- net BL: no longer U5.18 (GPIO18)
- net DC: no longer U5.14 (GPIO14)
- net GND: now also J4.2 (Pin_2)
- net MOSI: no longer U5.21 (GPIO21)
- net RST: no longer U5.15 (GPIO15)
- net RX1: now also J4.3 (Pin_3)
- net SCK: no longer U5.9 (GPIO9)
- net TX1: now also J4.4 (Pin_4)
- net VCC: now also J4.1 (Pin_1)
- no-connect marks 15 -> 12
Other:
- moved on the sheet: C4

Commit message: first order with cozir fix and i2c fix
Parts:
- removed D3: WS2812B, LED_SMD:LED_WS2812B-2020_PLCC4_2.0x2.0mm, symbol LED:WS2812B
- added F1: Polyfuse, Fuse:Fuse_Bourns_MF-RG300, symbol Device:Polyfuse
- added J5, J6: Conn_01x04, Connector_PinHeader_2.54mm:PinHeader_1x04_P2.54mm_Vertical, symbol Connector_Generic:Conn_01x04
Connections:
- net +3.3V: now also J5.2 (Pin_2), J6.2 (Pin_2)
- net CS: no longer U5.8 (GPIO8)
- net GND: now also J5.1 (Pin_1), J6.1 (Pin_1)
- net SCL: now also U5.21 (GPIO21); no longer U5.12 (GPIO12)
- net SDA: now also U5.22 (GPIO22); no longer U5.13 (GPIO13)
- net at PS1.1 (AC/L): now also F1.2
- net EX2: now reaches U5.14 (GPIO14)
- net EX2: now also J5.4 (Pin_4)
- net EX3: now reaches U5.15 (GPIO15)
- net EX3: now also J6.3 (Pin_3)
- net EX4: now reaches U5.18 (GPIO18)
- net EX4: now also J6.4 (Pin_4)
- net EX1: now reaches U5.9 (GPIO9)
- net EX1: now also J5.3 (Pin_3)
- no-connect marks 12 -> 14
