File: pcb/room-pcb.kicad_pcb (KiCad board)
At the start: 2 copper layers, 50 x 55 mm, 34 parts, among them J1 Conn_01x08, J2 Conn_01x02, J3 Conn_01x04, J4 Conn_01x05, J5 Conn_01x04, J6 Conn_01x04, U1 COZIR, U2 BH1750FVI-TR, U3 AHT20, U4 SCD41-D-R2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

Commit message: v4.1
Parts:
- TP1, TP2, TP3: footprint TestPoint:TestPoint_Loop_D2.60mm_Drill1.4mm_Beaded -> TestPoint:TestPoint_THTPad_D1.5mm_Drill0.7mm
Connections:
- J6 pad 3: EX3 -> MOSI
- J6 pad 4: EX4 -> SCK
- U5 pad 0: CAL -> unconnected-(U5-GPIO0-Pad0)
- U5 pad 14: EX2 -> SCK
- U5 pad 15: EX3 -> RST
- U5 pad 18: EX4 -> MOSI
- U5 pad 4: unconnected-(U5-GPIO4-Pad4) -> CAL
- U5 pad 5: unconnected-(U5-GPIO5-Pad5) -> CS
- U5 pad 8: unconnected-(U5-GPIO8-Pad8) -> EX1
- U5 pad 9: EX1 -> EX2
- U5 pad RX: unconnected-(U5-PadRX) -> BL
- U5 pad TX: unconnected-(U5-PadTX) -> DC
Routing:
- net +3.3V: track 0.00 -> 221.6 mm, vias 0 -> 6
- net VCC: track 0.00 -> 124.5 mm, vias 0 -> 2
- net SCL: track 0.00 -> 122.9 mm, vias 0 -> 6
- net SDA: track 0.00 -> 109.5 mm, vias 0 -> 5
- net GND: track 0.00 -> 54.1 mm, vias 0 -> 21
- net MOSI: track 0.00 -> 48.4 mm, vias 0 -> 3
- net RX: track 0.00 -> 46.3 mm, vias 0 -> 1
- net CLK: track 0.00 -> 46.1 mm, vias 0 -> 1
- net SCK: track 0.00 -> 45.5 mm, vias 0 -> 2
- net BAT+: track 0.00 -> 45.4 mm, vias 0 -> 1
- net WS: track 0.00 -> 43.4 mm
- net RX1: track 0.00 -> 42.6 mm, vias 0 -> 1
- net DATA: track 0.00 -> 41.4 mm
- net TX1: track 0.00 -> 40.5 mm, vias 0 -> 1
- net BAT-: track 0.00 -> 40.1 mm, vias 0 -> 1
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
Commit message: nice silk now
Parts:
- moved H1 1.23 mm to (139.9, 92.9)
- moved H2 1.23 mm to (104.8, 106.4)
- moved D1 0.82 mm to (136.4, 76.7)
- moved D2 0.68 mm to (139.7, 76.7)
Routing:
- net +3.3V: track 221.6 -> 223.1 mm
- net Net-(D1-DOUT): track 17.6 -> 18.3 mm
