File: pcb/_autosave-room-pcb.kicad_pcb (KiCad board)
At the start: 2 copper layers, 50 x 55 mm, 34 parts, among them J1 Conn_01x08, J2 Conn_01x02, J3 Conn_01x04, J4 Conn_01x05, J5 Conn_01x04, J6 Conn_01x04, U1 COZIR, U2 BH1750FVI-TR, U3 AHT20, U4 SCD41-D-R2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

Commit message: v4
Parts:
- TP1, TP2, TP3: footprint TestPoint:TestPoint_Loop_D2.60mm_Drill1.4mm_Beaded -> TestPoint:TestPoint_THTPad_D1.5mm_Drill0.7mm
- moved D2 0.58 mm to (139.8, 76.7)
- moved D1 0.51 mm to (136.1, 76.8), turned to -90 degrees
Connections:
- J6 pad 3: EX3 -> MOSI
- J6 pad 4: EX4 -> SCK
- U5 pad 0: CAL -> unconnected-(U5-GPIO0-Pad0)
- U5 pad 14: EX2 -> SCK
- U5 pad 15: EX3 -> RST
- U5 pad 18: EX4 -> MOSI
- U5 pad 4: unconnected-(U5-GPIO4-Pad4) -> CAL
- U5 pad 5: unconnected-(U5-GPIO5-Pad5) -> CS
- U5 pad 8: unconnected-(U5-GPIO8-Pad8) -> EX1
- U5 pad 9: EX1 -> EX2
- U5 pad RX: unconnected-(U5-PadRX) -> BL
- U5 pad TX: unconnected-(U5-PadTX) -> DC
Routing:
- net +3.3V: track 0.00 -> 243.1 mm, vias 0 -> 5
- net SDA: track 0.00 -> 116.1 mm, vias 0 -> 6
- net SCL: track 0.00 -> 109.2 mm, vias 0 -> 3
- net VCC: track 0.00 -> 95.2 mm, vias 0 -> 2
- net WS: track 0.00 -> 60.6 mm, vias 0 -> 2
- net CLK: track 0.00 -> 60.0 mm, vias 0 -> 3
- net MOSI: track 0.00 -> 50.7 mm, vias 0 -> 1
- net GND: track 0.00 -> 46.9 mm, vias 0 -> 28
- net SCK: track 0.00 -> 46.8 mm, vias 0 -> 4
- net BAT+: track 0.00 -> 46.6 mm, vias 0 -> 2
- net RX1: track 0.00 -> 45.3 mm, vias 0 -> 1
- net TX1: track 0.00 -> 42.5 mm, vias 0 -> 1
- net DATA: track 0.00 -> 41.4 mm
- net BAT-: track 0.00 -> 39.3 mm, vias 0 -> 1
- net EX1: track 0.00 -> 38.8 mm, vias 0 -> 1
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