File: pcb/room-pcb.kicad_sch (KiCad schematic)
At the start: 30 parts, among them J1 Conn_01x08, J2 Conn_01x02, J3 Conn_01x04, J4 Conn_01x05, J5 Conn_01x04, J6 Conn_01x04, U1 COZIR, U2 BH1750FVI-TR, U3 AHT20, U5 ESP32-C6_SUPERMINI_TH

Commit message: v3
Parts:
- added TP1, TP2, TP3: TestPoint, TestPoint:TestPoint_Loop_D2.60mm_Drill1.4mm_Beaded, symbol Connector:TestPoint
- D1, D2: symbol LED:WS2812B -> LED:WS2812B-2020
Connections:
- net +3.3V: now also D1.4 (VDD), D2.4 (VDD), TP3.1; no longer D1.1 (VDD), D2.1 (VDD)
- net GND: now also D1.2 (VSS), D2.2 (VSS), TP2.1; no longer D1.3 (VSS), D2.3 (VSS)
- net NEO: now also D1.3 (DIN); no longer D1.4 (DIN)
- net VCC: now also TP1.1
- new net: D1.1 (DOUT), D2.3 (DIN)
Changed lines of the file:
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@@
 	)
 	(junction
+		(at 43.18 29.21)
+		(diameter 0)
+		(color 0 0 0 0)
+	)
+	(junction
 		(at 274.32 114.3)
 		(diameter 0)
@@
 	)
 	(junction
+		(at 43.18 24.13)
+		(diameter 0)
+		(color 0 0 0 0)
+	)
+	(junction
 		(at 228.6 30.48)
 		(diameter 0)
@@
 	)
 	(junction
+		(at 72.39 78.74)
+		(diameter 0)
+		(color 0 0 0 0)
+	)
+	(junction
 		(at 173.99 80.01)
 		(diameter 0)
@@
 	)
 	(symbol
+		(lib_id "Connector:TestPoint")
+		(at 72.39 78.74 270)
+		(unit 1)
+		(exclude_from_sim no)
+		(in_bom yes)
+		(on_board yes)
+		(dnp no)
+		(fields_autoplaced yes)
+		(property "Reference" "TP3"
+			(at 77.47 77.4699 90)
+			(effects
+				(font
+					(size 1.27 1.27)
+				)
+				(justify left)
+			)
+		)
+		(property "Value" "TestPoint"
+			(at 77.47 80.0099 90)
+			(effects
+				(font
+					(size 1.27 1.27)
+				)
+				(justify left)
+			)
+		)
+		(property "Footprint" "TestPoint:TestPoint_Loop_D2.60mm_Drill1.4mm_Beaded"
+			(at 72.39 83.82 0)
+			(effects
+				(font
+					(size 1.27 1.27)
+				)
+				(hide yes)
+			)
+		)
+		(property "Datasheet" "~"
+			(at 72.39 83.82 0)
+			(effects
+				(font
+					(size 1.27 1.27)
+				)
+				(hide yes)
+			)
+		)
+		(property "Description" "test point"
+			(at 72.39 78.74 0)
+			(effects
+				(font
+					(size 1.27 1.27)
+				)
+				(hide yes)
+			)
+		)
+		(pin "1"
+		)
+		(instances
+			(project "room-pcb"
+				(path "/e86757dd-dfd1-45ab-bb50-15759bddd4c1"
+					(reference "TP3")
+					(unit 1)
+				)
+			)
+		)
+	)
+	(symbol
 		(lib_id "power:+3.3V")
 		(at 124.46 80.01 0)
@@
 	)
 	(symbol
+		(lib_id "Connector:TestPoint")
+		(at 43.18 29.21 270)
+		(unit 1)
+		(exclude_from_sim no)
+		(in_bom yes)
+		(on_board yes)
+		(dnp no)
+		(fields_autoplaced yes)
+		(property "Reference" "TP2"
+			(at 48.26 27.9399 90)
+			(effects
+				(font
+					(size 1.27 1.27)
+				)
+				(justify left)
+			)
+		)
+		(property "Value" "TestPoint"
+			(at 48.26 30.4799 90)
+			(effects
+				(font
+					(size 1.27 1.27)
+				)
+				(justify left)
+			)
+		)
+		(property "Footprint" "TestPoint:TestPoint_Loop_D2.60mm_Drill1.4mm_Beaded"
+			(at 43.18 34.29 0)
+			(effects
+				(font
+					(size 1.27 1.27)
+				)
+				(hide yes)
+			)
+		)
+		(property "Datasheet" "~"
+			(at 43.18 34.29 0)
+			(effects
+				(font
+					(size 1.27 1.27)
+				)
+				(hide yes)
+			)
+		)
+		(property "Description" "test point"
+			(at 43.18 29.21 0)
+			(effects
+				(font
+					(size 1.27 1.27)
+				)
+				(hide yes)
+			)
+		)
+		(pin "1"
+		)
+		(instances
+			(project "room-pcb"
+				(path "/e86757dd-dfd1-45ab-bb50-15759bddd4c1"
+					(reference "TP2")
+					(unit 1)
+				)
+			)
+		)
+	)
+	(symbol
 		(lib_id "power:VCC")
 		(at 43.18 24.13 0)
@@
 	)
 	(symbol
-		(lib_id "LED:WS2812B")
+		(lib_id "LED:WS2812B-2020")
 		(at 247.65 151.13 0)
 		(unit 1)
@@
 			)
 		)
-		(property "Datasheet" "https://cdn-shop.adafruit.com/datasheets/WS2812B.pdf"
+		(property "Datasheet" "https://cdn-shop.adafruit.com/product-files/4684/4684_WS2812B-2020_V1.3_EN.pdf"
 			(at 250.19 160.655 0)
 			(effects
@@
 			)
 		)
-		(property "Description" "RGB LED with integrated controller"
+		(property "Description" "RGB LED with integrated controller, 2.0 x 2.0 mm, 12 mA"
 			(at 247.65 151.13 0)
 			(effects
@@
 	)
 	(symbol
-		(lib_id "LED:WS2812B")
+		(lib_id "LED:WS2812B-2020")
 		(at 229.87 151.13 0)
 		(unit 1)
@@
 			)
 		)
-		(property "Datasheet" "https://cdn-shop.adafruit.com/datasheets/WS2812B.pdf"
+		(property "Datasheet" "https://cdn-shop.adafruit.com/product-files/4684/4684_WS2812B-2020_V1.3_EN.pdf"
 			(at 232.41 160.655 0)
 			(effects
@@
 			)
 		)
-		(property "Description" "RGB LED with integrated controller https://www.lcsc.com/product-detail/C965555.html?s_z=n_ws2812b"
+		(property "Description" "RGB LED with integrated controller, 2.0 x 2.0 mm, 12 mA"
 			(at 229.87 151.13 0)
 			(effects
@@
 					(unit 1)
 				)
+			)
+		)
+	)
+	(symbol
+		(lib_id "Connector:TestPoint")
+		(at 43.18 24.13 270)
+		(unit 1)
+		(exclude_from_sim no)
+		(in_bom yes)
+		(on_board yes)
+		(dnp no)
+		(fields_autoplaced yes)
+		(property "Reference" "TP1"
+			(at 48.26 22.8599 90)
+			(effects
+				(font
+					(size 1.27 1.27)
+				)
+				(justify left)
+			)
+		)
+		(property "Value" "TestPoint"
+			(at 48.26 25.3999 90)
+			(effects
+				(font
+					(size 1.27 1.27)
+				)
+				(justify left)
+			)
+		)
+		(property "Footprint" "TestPoint:TestPoint_Loop_D2.60mm_Drill1.4mm_Beaded"
+			(at 43.18 29.21 0)
+			(effects
+				(font
+					(size 1.27 1.27)
+				)
+				(hide yes)
+			)
+		)
+		(property "Datasheet" "~"
+			(at 43.18 29.21 0)
+			(effects
+				(font
+					(size 1.27 1.27)
+				)
+				(hide yes)
+			)
+		)
+		(property "Description" "test point"
+			(at 43.18 24.13 0)
+			(effects
+				(font
+					(size 1.27 1.27)
+				)
+				(hide yes)
+			)
+		)
+		(pin "1"
+		)
+		(instances
+			(project ""
+				(path "/e86757dd-dfd1-45ab-bb50-15759bddd4c1"
+					(reference "TP1")
+					(unit 1)
+				)

Commit message: v4
Parts:
- added U4: SCD41-D-R2, Sensor:Sensirion_SCD4x-1EP_10.1x10.1mm_P1.25mm_EP4.8x4.8mm, symbol Sensor_Gas:SCD41-D-R2
- C2, MK1, R2, R3, R4: now not fitted; now left out of the parts list
- TP1, TP2, TP3: footprint TestPoint:TestPoint_Loop_D2.60mm_Drill1.4mm_Beaded -> TestPoint:TestPoint_THTPad_D1.5mm_Drill0.7mm
Connections:
- net +3.3V: now also U4.19 (VDD), U4.7 (VDD)
- net BL: now also U5.RX
- net CAL: now also U5.4 (GPIO4); no longer U5.0 (GPIO0)
- net CS: now also U5.5 (GPIO5)
- net DC: now also U5.TX
- net EX1: now also U5.8 (GPIO8); no longer U5.9 (GPIO9)
- net EX2: now also U5.9 (GPIO9); no longer U5.14 (GPIO14)
- net GND: now also U4.20 (GND), U4.21 (GND), U4.6 (GND)
- net MOSI: now also J6.3 (Pin_3), U5.18 (GPIO18)
- net RST: now also U5.15 (GPIO15)
- net SCK: now also J6.4 (Pin_4), U5.14 (GPIO14)
- net SCL: now also U4.9 (SCL)
- net SDA: now also U4.10 (SDA)
- removed net EX3: J6.3 (Pin_3), U5.15 (GPIO15)
- removed net EX4: J6.4 (Pin_4), U5.18 (GPIO18)
- no-connect marks 14 -> 10
Other:
- note added: "gpio16 % 17"
- note added: "usb plus and minus"
